File: matrix.sch (KiCad schematic (older format))
At the start: 159 parts

Commit message: Schematic Finished
Parts:
- D1, D10, D11, D12, D13, D14, D15, D16, D17, D18, D19, D2, D20, D21, D22, D23, D24, D25, D26, D27, D28, D29, D3, D30, D31, D32, D33, D34, D35, D36, D37, D38, D39, D4, D40, D41, D42, D43, D44, D45, D46, D47, D48, D49, D5, D50, D51, D52, D53, D54, D55, D56, D57, D58, D59, D6, D60, D61, D62, D63, D64, D65, D66, D67, D68, D69, D7, D70, D71, D72, D73, D74, D75, D8, D9: renamed from D?; footprint (none) -> Diode_SMD:D_SOD-123
- K1, K10, K11, K12, K13, K14, K15, K17, K18, K19, K2, K21, K22, K23, K24, K25, K26, K27, K28, K29, K3, K30, K31, K32, K34, K37, K39, K4, K40, K41, K42, K43, K44, K45, K46, K47, K48, K49, K5, K50, K52, K54, K56, K57, K58, K59, K6, K60, K61, K62, K63, K64, K65, K66, K68, K69, K7, K71, K75, K8, K82, K83, K84, K9: renamed from K?; footprint (none) -> MX_Only:MXOnly-1U-NoLED
- K16: renamed from K?; footprint (none) -> MX_Only:MXOnly-2U-NoLED
- K20, K33, K78, K81: renamed from K?; footprint (none) -> MX_Only:MXOnly-1.5U-NoLED
- K35, K53, K70, K72, K74, K76, K77, K80: renamed from K?; footprint (none) -> MX_Only:MXOnly-1.25U-NoLED
- K36: renamed from K?; footprint (none) -> MX_Only:MXOnly-ISO-NoLED
- K38, K67: renamed from K?; footprint (none) -> MX_Only:MXOnly-1.75U-NoLED
- K51, K55: renamed from K?; footprint (none) -> MX_Only:MXOnly-2.25U-NoLED
- K73: renamed from K?; footprint (none) -> MX_Only:MXOnly-6.25U-NoLED
- K79: renamed from K?; footprint (none) -> MX_Only:MXOnly-7U-NoLED

Commit message: PCB Preparations Finished
routing time
so fun
Parts:
- K76: footprint MX_Only:MXOnly-1.25U-NoLED -> MX_Only:MXOnly-1.5U-NoLED
Changed lines of the file:
@@
 F 0 "K76" H 3250 7133 60  0000 C CNN
 F 1 "keyboard_parts_KEYSW" H 3250 6800 60  0001 C CNN
-F 2 "MX_Only:MXOnly-1.25U-NoLED" H 3250 6900 60  0001 C CNN
+F 2 "MX_Only:MXOnly-1.5U-NoLED" H 3250 6900 60  0001 C CNN
 F 3 "" H 3250 6900 60  0000 C CNN
 	1    3250 6900

Commit message: save
Parts:
- K73: footprint MX_Only:MXOnly-6.25U-NoLED -> MX_Only:MXOnly-6.25U-ReversedStabilizers-NoLED
- K79: footprint MX_Only:MXOnly-7U-NoLED -> MX_Only:MXOnly-7U-ReversedStabilizers-NoLED
Changed lines of the file:
@@
 F 0 "K79" H 7250 7133 60  0000 C CNN
 F 1 "keyboard_parts_KEYSW" H 7250 6800 60  0001 C CNN
-F 2 "MX_Only:MXOnly-7U-NoLED" H 7250 6900 60  0001 C CNN
+F 2 "MX_Only:MXOnly-7U-ReversedStabilizers-NoLED" H 7250 6900 60  0001 C CNN
 F 3 "" H 7250 6900 60  0000 C CNN
 	1    7250 6900
@@
 F 0 "K73" H 7250 6933 60  0000 C CNN
 F 1 "keyboard_parts_KEYSW" H 7250 6600 60  0001 C CNN
-F 2 "MX_Only:MXOnly-6.25U-NoLED" H 7250 6700 60  0001 C CNN
+F 2 "MX_Only:MXOnly-6.25U-ReversedStabilizers-NoLED" H 7250 6700 60  0001 C CNN
 F 3 "" H 7250 6700 60  0000 C CNN
 	1    7250 6700

Commit message: Rough Draft Finished
Connections:
- net at D70.2 (A), K79.2: now also K73.2
Changed lines of the file:
@@
 Wire Wire Line
 	9950 4100 9950 3500
+Wire Wire Line
+	6950 6700 6950 6900
+Connection ~ 6950 6900
 $EndSCHEMATC
