File: attempt2-pcb.kicad_pcb (KiCad board)
At the start: 2 copper layers, 174 parts, among them J1 Conn_01x04, K1 keyboard_parts_KEYSW, K10 keyboard_parts_KEYSW, K11 keyboard_parts_KEYSW, K12 keyboard_parts_KEYSW, K13 keyboard_parts_KEYSW, K14 keyboard_parts_KEYSW, K15 keyboard_parts_KEYSW, K16 keyboard_parts_KEYSW, K17 keyboard_parts_KEYSW, K18 keyboard_parts_KEYSW, K19 keyboard_parts_KEYSW, K2 keyboard_parts_KEYSW, K20 keyboard_parts_KEYSW, K21 keyboard_parts_KEYSW, K22 keyboard_parts_KEYSW, K23 keyboard_parts_KEYSW, K24 keyboard_parts_KEYSW, K25 keyboard_parts_KEYSW, K26 keyboard_parts_KEYSW, K27 keyboard_parts_KEYSW, K28 keyboard_parts_KEYSW, K29 keyboard_parts_KEYSW, K3 keyboard_parts_KEYSW, K30 keyboard_parts_KEYSW, K31 keyboard_parts_KEYSW, K32 keyboard_parts_KEYSW, K33 keyboard_parts_KEYSW, K34 keyboard_parts_KEYSW, K35 keyboard_parts_KEYSW, K36 keyboard_parts_KEYSW, K37 keyboard_parts_KEYSW, K38 keyboard_parts_KEYSW, K39 keyboard_parts_KEYSW, K4 keyboard_parts_KEYSW, K40 keyboard_parts_KEYSW, K41 keyboard_parts_KEYSW, K42 keyboard_parts_KEYSW, K43 keyboard_parts_KEYSW, K44 keyboard_parts_KEYSW, K45 keyboard_parts_KEYSW, K46 keyboard_parts_KEYSW, K47 keyboard_parts_KEYSW, K48 keyboard_parts_KEYSW, K49 keyboard_parts_KEYSW, K5 keyboard_parts_KEYSW, K50 keyboard_parts_KEYSW, K51 keyboard_parts_KEYSW, K52 keyboard_parts_KEYSW, K53 keyboard_parts_KEYSW, K54 keyboard_parts_KEYSW, K55 keyboard_parts_KEYSW, K56 keyboard_parts_KEYSW, K57 keyboard_parts_KEYSW, K58 keyboard_parts_KEYSW, K59 keyboard_parts_KEYSW, K6 keyboard_parts_KEYSW, K60 keyboard_parts_KEYSW, K61 keyboard_parts_KEYSW, K62 keyboard_parts_KEYSW, K63 keyboard_parts_KEYSW, K64 keyboard_parts_KEYSW, K65 keyboard_parts_KEYSW, K66 keyboard_parts_KEYSW, K67 keyboard_parts_KEYSW, K68 keyboard_parts_KEYSW, K69 keyboard_parts_KEYSW, K7 keyboard_parts_KEYSW, K70 keyboard_parts_KEYSW, K71 keyboard_parts_KEYSW, K72 keyboard_parts_KEYSW, K73 keyboard_parts_KEYSW, K74 keyboard_parts_KEYSW, K75 keyboard_parts_KEYSW, K76 keyboard_parts_KEYSW, K77 keyboard_parts_KEYSW, K78 keyboard_parts_KEYSW, K79 keyboard_parts_KEYSW, K8 keyboard_parts_KEYSW, K80 keyboard_parts_KEYSW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

Commit message: PCB prep actually finished
Parts:
- added U2: SRV05-4, Package_TO_SOT_SMD:SOT-23-6, B.Cu at (117.3, 59.6)
- C1, C2, C3, C4, C5, C6, C7, J1, R1, R2, R3, R4, SW1, U1, Y1: moved to B.Cu
- moved J1 110.5 mm to (143.5, 59.6), turned to 270 degrees
- moved C2 101.9 mm to (115.2, 74.8), turned to 0 degrees
- moved Y1 97.8 mm to (115.2, 78.1)
- moved R3 95.0 mm to (112.6, 58.2)
- moved C1 93.7 mm to (115.2, 81.4), turned to 0 degrees
- moved R2 93.6 mm to (112.6, 61.0)
- moved R1 93.3 mm to (120.3, 77.2), turned to 90 degrees
- moved SW1 91.0 mm to (125.9, 78.0), turned to 180 degrees
- moved C3 83.2 mm to (102.7, 68.3), turned to 270 degrees
- moved C5 79.9 mm to (111.1, 75.3), turned to 270 degrees
- moved C4 77.4 mm to (106.4, 85.6)
- moved U1 71.9 mm to (102.9, 77.3), turned to 270 degrees
- moved C7 64.3 mm to (97.8, 69.1), turned to 180 degrees
- moved R4 59.7 mm to (100.1, 88.1), turned to 180 degrees
- moved C6 54.8 mm to (93.9, 78.7), turned to 0 degrees
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
Commit message: save
Parts:
- K73: footprint MX_Only:MXOnly-6.25U-NoLED -> MX_Only:MXOnly-6.25U-ReversedStabilizers-NoLED
- K79: footprint MX_Only:MXOnly-7U-NoLED -> MX_Only:MXOnly-7U-ReversedStabilizers-NoLED
- moved U2 4.89 mm to (122.2, 59.5)
- moved C3 0.51 mm to (102.2, 68.3)
- moved R3 0.25 mm to (112.6, 58.4)
- moved R2 0.25 mm to (112.6, 60.7)
Routing:
- net GND: track 0.00 -> 129.0 mm, vias 0 -> 4
- net +5V: track 0.00 -> 76.4 mm, vias 0 -> 6
- net D-: track 0.00 -> 26.6 mm
- net D+: track 0.00 -> 26.6 mm
- net Net-(R1-Pad2): track 0.00 -> 24.5 mm
- net Net-(R3-Pad1): track 0.00 -> 19.4 mm
- net VBUS: track 0.00 -> 18.4 mm
- net Net-(R2-Pad1): track 0.00 -> 17.9 mm
- net Net-(C1-Pad1): track 0.00 -> 11.5 mm
- net Net-(C2-Pad1): track 0.00 -> 9.34 mm
- net Net-(R4-Pad2): track 0.00 -> 5.23 mm
- net Net-(C3-Pad1): track 0.00 -> 4.94 mm
Other:
- board outline added: 328.6 x 95.3 mm
- net class Default: trace_width 0.25 -> 0.254
- net class Power added: clearance 0.2, trace_width 0.381, via_dia 0.8, via_drill 0.4

Commit message: Rough Draft Finished
Parts:
- moved D70 36.5 mm to (227.0, 126.2)
- moved D51 20.6 mm to (76.2, 107.2)
- moved D47 6.70 mm to (335.0, 81.4)
- moved D48 6.35 mm to (352.4, 88.1)
- moved D15 4.76 mm to (339.7, 54.8)
- moved R4 2.90 mm to (98.4, 90.5), turned to 90 degrees
- moved D32 1.59 mm to (360.4, 69.1)
- moved C6 0.63 mm to (93.2, 78.7)
Connections:
- K73 pad 2: Net-(K73-Pad2) -> Net-(D70-Pad2)
- U1 pad 1: Net-(U1-Pad1) -> Row0
- U1 pad 12: Net-(U1-Pad12) -> Row1
- U1 pad 18: Net-(U1-Pad18) -> Col16
- U1 pad 19: Net-(U1-Pad19) -> Col15
- U1 pad 20: Net-(U1-Pad20) -> Col14
- U1 pad 21: Net-(U1-Pad21) -> Col13
- U1 pad 22: Net-(U1-Pad22) -> Col12
- U1 pad 25: Net-(U1-Pad25) -> Col11
- U1 pad 26: Net-(U1-Pad26) -> Col10
- U1 pad 27: Net-(U1-Pad27) -> Col9
- U1 pad 28: Net-(U1-Pad28) -> Col8
- U1 pad 29: Net-(U1-Pad29) -> Col7
- U1 pad 30: Net-(U1-Pad30) -> Col6
- U1 pad 31: Net-(U1-Pad31) -> Col5
- U1 pad 32: Net-(U1-Pad32) -> Col4
- U1 pad 36: Net-(U1-Pad36) -> Row2
- U1 pad 37: Net-(U1-Pad37) -> Col0
- U1 pad 38: Net-(U1-Pad38) -> Col1
- U1 pad 39: Net-(U1-Pad39) -> Row3
- U1 pad 40: Net-(U1-Pad40) -> Row4
- U1 pad 41: Net-(U1-Pad41) -> Col3
Routing:
- net Row4: track 0.00 -> 379.0 mm, vias 0 -> 2
- net Col15: track 0.00 -> 378.1 mm
- net Col14: track 0.00 -> 368.5 mm
- net Row2: track 0.00 -> 367.8 mm, vias 0 -> 2
- net Row3: track 0.00 -> 364.4 mm, vias 0 -> 2
- net Row0: track 0.00 -> 344.4 mm, vias 0 -> 2
- net Col13: track 0.00 -> 327.0 mm
- net Row1: track 0.00 -> 323.3 mm, vias 0 -> 2
- net Col16: track 0.00 -> 319.8 mm, vias 0 -> 4
- net Col12: track 0.00 -> 304.7 mm
- net Col11: track 0.00 -> 285.6 mm
- net Col10: track 0.00 -> 245.1 mm
- net Col9: track 0.00 -> 225.7 mm
- net Col6: track 0.00 -> 212.1 mm
- net Col8: track 0.00 -> 207.0 mm
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
Commit message: Fill Zones
Routing:
- added copper zone on B.Cu, net GND
Changed lines of the file:
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@@
   (segment (start 98.87 89.105) (end 98.425 89.55) (width 0.254) (layer B.Cu) (net 109))
   (segment (start 98.87 83.043) (end 98.87 89.105) (width 0.254) (layer B.Cu) (net 109))
+  (zone (net 1) (net_name GND) (layer B.Cu) (hatch edge 0.508)
+    (connect_pads (clearance 0.508))
+    (min_thickness 0.254)
+    (fill yes (arc_segments 32) (thermal_gap 0.508) (thermal_bridge_width 0.508))
+    (polygon
+      (pts
+        (xy 98.425 73.025) (xy 107.15625 73.025) (xy 107.15625 81.75625) (xy 98.425 81.75625)
+      )
+    )
+  )
+  (zone (net 1) (net_name GND) (layer B.Cu) (hatch edge 0.508)
+    (connect_pads (clearance 0.508))
+    (min_thickness 0.254)
+    (fill yes (arc_segments 32) (thermal_gap 0.508) (thermal_bridge_width 0.508))
+    (polygon
+      (pts
+        (xy 113.411 73.787) (xy 116.967 73.787) (xy 117.348 76.327) (xy 117.348 79.883) (xy 116.967 82.423)
+        (xy 113.411 82.423) (xy 113.03 79.883) (xy 113.03 76.327)
+      )
+    )
+  )
 )

Commit message: proofing
Parts:
- SW1: value SW_Push -> Reset
Connections:
- net Net-(C1-Pad1) renamed XTAL1
- net Net-(C2-Pad1) renamed XTAL2
- net Net-(R1-Pad2) renamed Reset
- net Net-(R2-Pad1) renamed /MCU_D+
- net Net-(R3-Pad1) renamed /MCU_D-
- U1 pad 10: Net-(U1-Pad10) -> Col2
Routing:
- net Col2: track 89.4 -> 96.9 mm
- net Col14: track 368.5 -> 374.8 mm
- net /MCU_D+: track 17.9 -> 18.7 mm
