File: attempt2-pcb.kicad_pcb (KiCad board)
At the start: 2 copper layers, 328.6 x 95.3 mm, 175 parts, among them J1 Conn_01x04, K1 keyboard_parts_KEYSW, K10 keyboard_parts_KEYSW, K11 keyboard_parts_KEYSW, K12 keyboard_parts_KEYSW, K13 keyboard_parts_KEYSW, K14 keyboard_parts_KEYSW, K15 keyboard_parts_KEYSW, K16 keyboard_parts_KEYSW, K17 keyboard_parts_KEYSW, K18 keyboard_parts_KEYSW, K19 keyboard_parts_KEYSW, K2 keyboard_parts_KEYSW, K20 keyboard_parts_KEYSW, K21 keyboard_parts_KEYSW, K22 keyboard_parts_KEYSW, K23 keyboard_parts_KEYSW, K24 keyboard_parts_KEYSW, K25 keyboard_parts_KEYSW, K26 keyboard_parts_KEYSW, K27 keyboard_parts_KEYSW, K28 keyboard_parts_KEYSW, K29 keyboard_parts_KEYSW, K3 keyboard_parts_KEYSW, K30 keyboard_parts_KEYSW, K31 keyboard_parts_KEYSW, K32 keyboard_parts_KEYSW, K33 keyboard_parts_KEYSW, K34 keyboard_parts_KEYSW, K35 keyboard_parts_KEYSW, K36 keyboard_parts_KEYSW, K37 keyboard_parts_KEYSW, K38 keyboard_parts_KEYSW, K39 keyboard_parts_KEYSW, K4 keyboard_parts_KEYSW, K40 keyboard_parts_KEYSW, K41 keyboard_parts_KEYSW, K42 keyboard_parts_KEYSW, K43 keyboard_parts_KEYSW, K44 keyboard_parts_KEYSW, K45 keyboard_parts_KEYSW, K46 keyboard_parts_KEYSW, K47 keyboard_parts_KEYSW, K48 keyboard_parts_KEYSW, K49 keyboard_parts_KEYSW, K5 keyboard_parts_KEYSW, K50 keyboard_parts_KEYSW, K51 keyboard_parts_KEYSW, K52 keyboard_parts_KEYSW, K53 keyboard_parts_KEYSW, K54 keyboard_parts_KEYSW, K55 keyboard_parts_KEYSW, K56 keyboard_parts_KEYSW, K57 keyboard_parts_KEYSW, K58 keyboard_parts_KEYSW, K59 keyboard_parts_KEYSW, K6 keyboard_parts_KEYSW, K60 keyboard_parts_KEYSW, K61 keyboard_parts_KEYSW, K62 keyboard_parts_KEYSW, K63 keyboard_parts_KEYSW, K64 keyboard_parts_KEYSW, K65 keyboard_parts_KEYSW, K66 keyboard_parts_KEYSW, K67 keyboard_parts_KEYSW, K68 keyboard_parts_KEYSW, K69 keyboard_parts_KEYSW, K7 keyboard_parts_KEYSW, K70 keyboard_parts_KEYSW, K71 keyboard_parts_KEYSW, K72 keyboard_parts_KEYSW, K73 keyboard_parts_KEYSW, K74 keyboard_parts_KEYSW, K75 keyboard_parts_KEYSW, K76 keyboard_parts_KEYSW, K77 keyboard_parts_KEYSW, K78 keyboard_parts_KEYSW, K79 keyboard_parts_KEYSW, K8 keyboard_parts_KEYSW, K80 keyboard_parts_KEYSW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

Commit message: Big Changes
Parts:
- U1: value ATmega32U4-AU -> ATmega32U4-MU; footprint Package_QFP:TQFP-44_10x10mm_P0.8mm -> Package_DFN_QFN:QFN-44-1EP_7x7mm_P0.5mm_EP5.2x5.2mm
- moved U1 0.76 mm to (102.3, 77.9)
Routing:
- net +5V: track 78.2 -> 96.2 mm
- net GND: track 135.0 -> 139.2 mm
- net Row1: track 323.3 -> 327.3 mm
- net Reset: track 24.7 -> 28.6 mm
- net Col2: track 96.9 -> 100.5 mm
- net Col12: track 304.7 -> 308.0 mm
- net Row0: track 344.4 -> 347.7 mm
- net XTAL2: track 9.34 -> 12.6 mm
- net Col13: track 327.0 -> 330.2 mm
- net XTAL1: track 11.5 -> 14.6 mm
- net Net-(C3-Pad1): track 4.94 -> 8.05 mm
- net Col14: track 374.8 -> 377.9 mm
- net /MCU_D-: track 19.4 -> 22.5 mm
- net Col16: track 319.8 -> 322.8 mm
- net Col15: track 378.1 -> 381.1 mm
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- removed copper zone on B.Cu, net GND
Other:
- net class Power: trace_width 0.381 -> 0.254
