File: attempt2-pcb.sch (KiCad schematic (older format))
At the start: 160 parts

Commit message: Switch matrix save
Parts:
- removed D? (x71): SOD-123, symbol Device:D_Small
- removed MX? (x71): MX-NoLED, symbol MX_Alps_Hybrid:MX-NoLED
- added D? (x3): SOD_123, symbol Device:D_Small
- added MX? (x3): MX-NoLED, symbol MX_Alps_Hybrid:MX-NoLED
Connections:
- net labels removed: Col10, Col11, Col12, Col13, Col14, Col15, Col2, Col3, Col4, Col5, Col6, Col7, Col8, Col9, Row1, Row2, Row3, Row4
- wire segments 292 -> 61

Commit message: Switch matrix save
restarted and cleaned up matrix
added split backspace support
Parts:
- removed D? (x3): SOD_123, symbol Device:D_Small
- removed MX? (x3): MX-NoLED, symbol MX_Alps_Hybrid:MX-NoLED
- added D? (x17): SOD-123, symbol Device:D_Small
- added MX? (x18): MX-NoLED, symbol MX_Alps_Hybrid:MX-NoLED
Connections:
- net labels added: Col10, Col11, Col12, Col13, Col14, Col15, Col16, Col2, Col3, Col4, Col5, Col6, Col7, Col8, Col9
- wire segments 61 -> 110
Other:
- moved on the sheet: C?, R?, SW?, U?, Y?

Commit message: Switch Matrix Save
switch matrix almost done
Parts:
- removed D? (x17): SOD-123, symbol Device:D_Small
- removed MX? (x18): MX-NoLED, symbol MX_Alps_Hybrid:MX-NoLED
Connections:
- net labels removed: Col0, Col1, Col10, Col11, Col12, Col13, Col14, Col15, Col16, Col2, Col3, Col4, Col5, Col6, Col7, Col8, Col9, Row0
- wire segments 110 -> 50

Commit message: Schematic Finished
Parts:
- removed F?: 500mA, symbol Device:Polyfuse_Small
- removed J?: USB_C_Receptacle_USB2.0, symbol Connector:USB_C_Receptacle_USB2.0
- removed R? (x2): 5.1k, symbol Device:R_Small
- added J1: Conn_01x04, random-keyboard-parts:JST-SR-4, symbol Connector_Generic:Conn_01x04
- C1, C2, C3, C4, C5, C6, C7: renamed from C?; footprint (none) -> Capacitor_SMD:C_0805_2012Metric
- R1, R2, R3, R4: renamed from R?; footprint (none) -> Resistor_SMD:R_0805_2012Metric
- SW1: renamed from SW?; footprint (none) -> random-keyboard-parts:SKQG-1155865
- Y1: renamed from Y?; footprint (none) -> Crystal:Crystal_SMD_3225-4Pin_3.2x2.5mm
- gave numbers to parts that had none: 1
Connections:
- net D+: now also J1.3 (Pin_3)
- net D-: now also J1.2 (Pin_2)
- net GND: now also J1.4 (Pin_4)
- new net VBUS: J1.1 (Pin_1)
Changed lines of the file:
@@
 	2150 3900 2150 4150
 $Comp
-L Device:R_Small R?
+L Device:R_Small R1
 U 1 1 622EC068
 P 2150 3800
-F 0 "R?" H 2209 3846 50  0000 L CNN
+F 0 "R1" H 2209 3846 50  0000 L CNN
 F 1 "10k" H 2209 3755 50  0000 L CNN
-F 2 "" H 2150 3800 50  0001 C CNN
+F 2 "Resistor_SMD:R_0805_2012Metric" H 2150 3800 50  0001 C CNN
 F 3 "~" H 2150 3800 50  0001 C CNN
 	1    2150 3800
@@
 $EndComp
 $Comp
-L Switch:SW_Push SW?
+L Switch:SW_Push SW1
 U 1 1 622E5F62
 P 1850 4150
-F 0 "SW?" H 1850 4435 50  0000 C CNN
+F 0 "SW1" H 1850 4435 50  0000 C CNN
 F 1 "SW_Push" H 1850 4344 50  0000 C CNN
-F 2 "" H 1850 4350 50  0001 C CNN
+F 2 "random-keyboard-parts:SKQG-1155865" H 1850 4350 50  0001 C CNN
 F 3 "~" H 1850 4350 50  0001 C CNN
 	1    1850 4150
@@
 	1400 4600 1800 4600
 $Comp
-L Device:C_Small C?
+L Device:C_Small C2
 U 1 1 622D720B
 P 1300 4600
-F 0 "C?" V 1071 4600 50  0000 C CNN
+F 0 "C2" V 1071 4600 50  0000 C CNN
 F 1 "22pF" V 1162 4600 50  0000 C CNN
-F 2 "" H 1300 4600 50  0001 C CNN
+F 2 "Capacitor_SMD:C_0805_2012Metric" H 1300 4600 50  0001 C CNN
 F 3 "~" H 1300 4600 50  0001 C CNN
 	1    1300 4600
@@
 $EndComp
 $Comp
-L Device:C_Small C?
+L Device:C_Small C1
 U 1 1 622D5727
 P 1300 4300
-F 0 "C?" V 1071 4300 50  0000 C CNN
+F 0 "C1" V 1071 4300 50  0000 C CNN
 F 1 "22pF" V 1162 4300 50  0000 C CNN
-F 2 "" H 1300 4300 50  0001 C CNN
+F 2 "Capacitor_SMD:C_0805_2012Metric" H 1300 4300 50  0001 C CNN
 F 3 "~" H 1300 4300 50  0001 C CNN
 	1    1300 4300
@@
 	1800 4350 2250 4350
 $Comp
-L Device:Crystal_GND24_Small Y?
+L Device:Crystal_GND24_Small Y1
 U 1 1 622D2674
 P 1800 4450
-F 0 "Y?" V 1754 4594 50  0000 L CNN
+F 0 "Y1" V 1754 4594 50  0000 L CNN
 F 1 "16MHz" V 1845 4594 50  0000 L CNN
-F 2 "" H 1800 4450 50  0001 C CNN
+F 2 "Crystal:Crystal_SMD_3225-4Pin_3.2x2.5mm" H 1800 4450 50  0001 C CNN
 F 3 "~" H 1800 4450 50  0001 C CNN
 	1    1800 4450
@@
 	750  6400 1050 6400
 $Comp
-L Device:C_Small C?
+L Device:C_Small C4
 U 1 1 622A9F7D
 P 750 6500
-F 0 "C?" H 842 6546 50  0000 L CNN
+F 0 "C4" H 842 6546 50  0000 L CNN
 F 1 "0.1uF" H 842 6455 50  0000 L CNN
-F 2 "" H 750 6500 50  0001 C CNN
+F 2 "Capacitor_SMD:C_0805_2012Metric" H 750 6500 50  0001 C CNN
 F 3 "~" H 750 6500 50  0001 C CNN
 	1    750  6500
@@
 $EndComp
 $Comp
-L Device:C_Small C?
+L Device:C_Small C7
 U 1 1 622A8DF1
 P 1650 6500
-F 0 "C?" H 1742 6546 50  0000 L CNN
+F 0 "C7" H 1742 6546 50  0000 L CNN
 F 1 "10uF" H 1742 6455 50  0000 L CNN
-F 2 "" H 1650 6500 50  0001 C CNN
+F 2 "Capacitor_SMD:C_0805_2012Metric" H 1650 6500 50  0001 C CNN
 F 3 "~" H 1650 6500 50  0001 C CNN
 	1    1650 6500
@@
 $EndComp
 $Comp
-L Device:C_Small C?
+L Device:C_Small C6
 U 1 1 622A7C38
 P 1350 6500
-F 0 "C?" H 1442 6546 50  0000 L CNN
+F 0 "C6" H 1442 6546 50  0000 L CNN
 F 1 "0.1uF" H 1442 6455 50  0000 L CNN
-F 2 "" H 1350 6500 50  0001 C CNN
+F 2 "Capacitor_SMD:C_0805_2012Metric" H 1350 6500 50  0001 C CNN
 F 3 "~" H 1350 6500 50  0001 C CNN
 	1    1350 6500
@@
 $EndComp
 $Comp
-L Device:C_Small C?
+L Device:C_Small C5
 U 1 1 622A6EAD
 P 1050 6500
-F 0 "C?" H 1142 6546 50  0000 L CNN
+F 0 "C5" H 1142 6546 50  0000 L CNN
 F 1 "0.1uF" H 1142 6455 50  0000 L CNN
-F 2 "" H 1050 6500 50  0001 C CNN
+F 2 "Capacitor_SMD:C_0805_2012Metric" H 1050 6500 50  0001 C CNN
 F 3 "~" H 1050 6500 50  0001 C CNN
 	1    1050 6500
@@
 	1650 5450 2250 5450
 $Comp
-L Device:C_Small C?
+L Device:C_Small C3
 U 1 1 622990FF
 P 1650 5550
-F 0 "C?" H 1742 5596 50  0000 L CNN
+F 0 "C3" H 1742 5596 50  0000 L CNN
 F 1 "1uF" H 1742 5505 50  0000 L CNN
-F 2 "" H 1650 5550 50  0001 C CNN
+F 2 "Capacitor_SMD:C_0805_2012Metric" H 1650 5550 50  0001 C CNN
 F 3 "~" H 1650 5550 50  0001 C CNN
 	1    1650 5550
@@
 	1600 5150 2250 5150
 $Comp
-L Device:R_Small R?
+L Device:R_Small R3
 U 1 1 622967D3
 P 1150 5250
-F 0 "R?" V 954 5250 50  0000 C CNN
+F 0 "R3" V 954 5250 50  0000 C CNN
 F 1 "22" V 1045 5250 50  0000 C CNN
-F 2 "" H 1150 5250 50  0001 C CNN
+F 2 "Resistor_SMD:R_0805_2012Metric" H 1150 5250 50  0001 C CNN
 F 3 "~" H 1150 5250 50  0001 C CNN
 	1    1150 5250
@@
 $EndComp
 $Comp
-L Device:R_Small R?
+L Device:R_Small R2
 U 1 1 6229476D
 P 1500 5150
-F 0 "R?" V 1304 5150 50  0000 C CNN
+F 0 "R2" V 1304 5150 50  0000 C CNN
 F 1 "22" V 1395 5150 50  0000 C CNN
-F 2 "" H 1500 5150 50  0001 C CNN
+F 2 "Resistor_SMD:R_0805_2012Metric" H 1500 5150 50  0001 C CNN
 F 3 "~" H 1500 5150 50  0001 C CNN
 	1    1500 5150
@@
 	3450 6250 3700 6250
 $Comp
-L Device:R_Small R?
+L Device:R_Small R4
 U 1 1 6229109B
 P 3800 6250
-F 0 "R?" V 3604 6250 50  0000 C CNN
+F 0 "R4" V 3604 6250 50  0000 C CNN
 F 1 "10k" V 3695 6250 50  0000 C CNN
-F 2 "" H 3800 6250 50  0001 C CNN
+F 2 "Resistor_SMD:R_0805_2012Metric" H 3800 6250 50  0001 C CNN
 F 3 "~" H 3800 6250 50  0001 C CNN
 	1    3800 6250
@@
 $EndComp
 $Comp
-L MCU_Microchip_ATmega:ATmega32U4-AU U?
+L MCU_Microchip_ATmega:ATmega32U4-AU U1
 U 1 1 6227D02D
 P 2850 5650
-F 0 "U?" H 2850 3761 50  0000 C CNN
+F 0 "U1" H 2850 3761 50  0000 C CNN
 F 1 "ATmega32U4-AU" H 2850 3670 50  0000 C CNN
 F 2 "Package_QFP:TQFP-44_10x10mm_P0.8mm" H 2850 5650 50  0001 C CIN
@@
 	1    0    0    -1
 $EndComp
-$Comp
-L power:+5V #PWR0111
-U 1 1 6231E86A
-P 3200 1100
-F 0 "#PWR0111" H 3200 950 50  0001 C CNN
-F 1 "+5V" H 3215 1273 50  0000 C CNN
-F 2 "" H 3200 1100 50  0001 C CNN
-F 3 "" H 3200 1100 50  0001 C CNN
-	1    3200 1100
-	1    0    0    -1
-$EndComp
-Wire Wire Line
-	1300 2700 1300 2600
-$Comp
-L power:GND #PWR0112
-U 1 1 62333235
-P 1300 2700
-F 0 "#PWR0112" H 1300 2450 50  0001 C CNN
-F 1 "GND" H 1305 2527 50  0000 C CNN
-F 2 "" H 1300 2700 50  0001 C CNN
-F 3 "" H 1300 2700 50  0001 C CNN
-	1    1300 2700
-	1    0    0    -1
-$EndComp
-Text GLabel 1900 1800 2    50   Input ~ 0
-D+
-Text GLabel 1900 1700 2    50   Input ~ 0
-D-
-Wire Wire Line
-	1900 1900 1900 1800
-Wire Wire Line
-	1900 1600 1900 1700
-Wire Wire Line
-	1900 1400 2400 1400
-$Comp
-L power:GND #PWR0113
-U 1 1 623286EB
-P 2600 1400
-F 0 "#PWR0113" H 2600 1150 50  0001 C CNN
-F 1 "GND" V 2605 1272 50  0000 R CNN
-F 2 "" H 2600 1400 50  0001 C CNN
-F 3 "" H 2600 1400 50  0001 C CNN
-	1    2600 1400
-	0    -1   -1   0
-$EndComp
-$Comp
-L Device:R_Small R?
-U 1 1 62327EEE
-P 2500 1400
-F 0 "R?" V 2696 1400 50  0000 C CNN
-F 1 "5.1k" V 2605 1400 50  0000 C CNN
-F 2 "" H 2500 1400 50  0001 C CNN
-F 3 "~" H 2500 1400 50  0001 C CNN
-	1    2500 1400
-	0    -1   -1   0
-$EndComp
-$Comp
-L power:GND #PWR0114
-U 1 1 62324CC0
-P 2100 1300
-F 0 "#PWR0114" H 2100 1050 50  0001 C CNN
-F 1 "GND" V 2105 1172 50  0000 R CNN
-F 2 "" H 2100 1300 50  0001 C CNN
-F 3 "" H 2100 1300 50  0001 C CNN
-	1    2100 1300
-	0    -1   -1   0
-$EndComp
-$Comp
-L Device:R_Small R?
-U 1 1 62323CF0
-P 2000 1300
-F 0 "R?" V 2196 1300 50  0000 C CNN
-F 1 "5.1k" V 2105 1300 50  0000 C CNN
-F 2 "" H 2000 1300 50  0001 C CNN
-F 3 "~" H 2000 1300 50  0001 C CNN
-	1    2000 1300
-	0    -1   -1   0
-$EndComp
-Wire Wire Line
-	2150 1100 1900 1100
-$Comp
-L power:VCC #PWR0115
-U 1 1 623224A8
-P 2150 1100
-F 0 "#PWR0115" H 2150 950 50  0001 C CNN
-F 1 "VCC" H 2167 1273 50  0000 C CNN
-F 2 "" H 2150 1100 50  0001 C CNN
-F 3 "" H 2150 1100 50  0001 C CNN
-	1    2150 1100
-	1    0    0    -1
-$EndComp
-Connection ~ 2150 1100
-Wire Wire Line
-	2450 1100 2150 1100
-Wire Wire Line
-	3200 1100 2650 1100
-$Comp
-L Device:Polyfuse_Small F?
-U 1 1 6231CA3D
-P 2550 1100
-F 0 "F?" V 2345 1100 50  0000 C CNN
-F 1 "500mA" V 2436 1100 50  0000 C CNN
-F 2 "" H 2600 900 50  0001 L CNN
-F 3 "~" H 2550 1100 50  0001 C CNN
-	1    2550 1100
-	0    1    1    0
-$EndComp
-$Comp
-L Connector:USB_C_Receptacle_USB2.0 J?
-U 1 1 62313A71
-P 1300 1700
-F 0 "J?" H 1407 2567 50  0000 C CNN
-F 1 "USB_C_Receptacle_USB2.0" H 1407 2476 50  0000 C CNN
-F 2 "" H 1450 1700 50  0001 C CNN
-F 3 "https://www.usb.org/sites/default/files/documents/usb_type-c.zip" H 1450 1700 50  0001 C CNN
-	1    1300 1700
-	1    0    0    -1
-$EndComp
 $Sheet
-S 6850 4350 1600 1450
+S 9500 4950 1600 1450
 U 62363975
 F0 "switch matrix" 50
 F1 "matrix.sch" 50
 $EndSheet
+$Comp
+L Connector_Generic:Conn_01x04 J1
+U 1 1 626DFEAA
+P 1400 2250
+F 0 "J1" H 1480 2242 50  0000 L CNN
+F 1 "Conn_01x04" H 1480 2151 50  0000 L CNN
+F 2 "random-keyboard-parts:JST-SR-4" H 1400 2250 50  0001 C CNN
+F 3 "~" H 1400 2250 50  0001 C CNN
+	1    1400 2250
+	1    0    0    -1
+$EndComp
+Wire Wire Line
+	1200 2150 1050 2150
+Wire Wire Line
+	1050 2150 1050 2050
+$Comp
+L power:VBUS #PWR0111
+U 1 1 626E380F
+P 1050 2050
+F 0 "#PWR0111" H 1050 1900 50  0001 C CNN
+F 1 "VBUS" H 1065 2223 50  0000 C CNN
+F 2 "" H 1050 2050 50  0001 C CNN
+F 3 "" H 1050 2050 50  0001 C CNN
+	1    1050 2050
+	1    0    0    -1
+$EndComp
+Wire Wire Line
+	1200 2450 1050 2450
+Wire Wire Line
+	1050 2450 1050 2550
+$Comp
+L power:GND #PWR0112
+U 1 1 626E5F38
+P 1050 2550
+F 0 "#PWR0112" H 1050 2300 50  0001 C CNN
+F 1 "GND" H 1055 2377 50  0000 C CNN
+F 2 "" H 1050 2550 50  0001 C CNN
+F 3 "" H 1050 2550 50  0001 C CNN
+	1    1050 2550
+	1    0    0    -1
+$EndComp
+Wire Wire Line
+	1200 2350 1050 2350
+Wire Wire Line
+	1200 2250 1050 2250
+Text GLabel 1050 2250 0    50   Input ~ 0
+D-
+Text GLabel 1050 2350 0    50   Input ~ 0
+D+
 $EndSCHEMATC

Commit message: PCB prep actually finished
Parts:
- added U2: SRV05-4, Package_TO_SOT_SMD:SOT-23-6, symbol Power_Protection:SRV05-4
Connections:
- net D+: now also U2.1 (IO1)
- net D-: now also U2.6 (IO4)
- net GND: now also U2.2 (VN)
- net VBUS: now also U2.5 (VP)
- no-connect marks 0 -> 2
Changed lines of the file:
@@
 Text GLabel 1050 2350 0    50   Input ~ 0
 D+
+$Comp
+L Power_Protection:SRV05-4 U2
+U 1 1 6234A89E
+P 3300 1800
+F 0 "U2" H 3300 2481 50  0000 C CNN
+F 1 "SRV05-4" H 3300 2390 50  0000 C CNN
+F 2 "Package_TO_SOT_SMD:SOT-23-6" H 4000 1350 50  0001 C CNN
+F 3 "http://www.onsemi.com/pub/Collateral/SRV05-4-D.PDF" H 3300 1800 50  0001 C CNN
+	1    3300 1800
+	1    0    0    -1
+$EndComp
+NoConn ~ 3800 1700
+NoConn ~ 2800 1900
+Wire Wire Line
+	2800 1700 2650 1700
+Wire Wire Line
+	3800 1900 3950 1900
+Text GLabel 2650 1700 0    50   Input ~ 0
+D+
+Text GLabel 3950 1900 2    50   Input ~ 0
+D-
+Wire Wire Line
+	3300 2300 3550 2300
+$Comp
+L power:GND #PWR0113
+U 1 1 623564EB
+P 3550 2300
+F 0 "#PWR0113" H 3550 2050 50  0001 C CNN
+F 1 "GND" H 3555 2127 50  0000 C CNN
+F 2 "" H 3550 2300 50  0001 C CNN
+F 3 "" H 3550 2300 50  0001 C CNN
+	1    3550 2300
+	1    0    0    -1
+$EndComp
+Wire Wire Line
+	3300 1300 3550 1300
+$Comp
+L power:VBUS #PWR0114
+U 1 1 6235878A
+P 3550 1300
+F 0 "#PWR0114" H 3550 1150 50  0001 C CNN
+F 1 "VBUS" H 3565 1473 50  0000 C CNN
+F 2 "" H 3550 1300 50  0001 C CNN
+F 3 "" H 3550 1300 50  0001 C CNN
+	1    3550 1300
+	1    0    0    -1
+$EndComp
 $EndSCHEMATC

Commit message: Rough Draft Finished
Connections:
- net Row0: now reaches U1.1 (PE6)
- net Row1: now reaches U1.12 (PB7)
- net Col16: now reaches U1.18 (PD0)
- net Col15: now reaches U1.19 (PD1)
- net Col14: now reaches U1.20 (PD2)
- net Col13: now reaches U1.21 (PD3)
- net Col12: now reaches U1.22 (PD5)
- net Col11: now reaches U1.25 (PD4)
- net Col10: now reaches U1.26 (PD6)
- net Col9: now reaches U1.27 (PD7)
- net Col8: now reaches U1.28 (PB4)
- net Col7: now reaches U1.29 (PB5)
- net Col6: now reaches U1.30 (PB6)
- net Col5: now reaches U1.31 (PC6)
- net Col4: now reaches U1.32 (PC7)
- net Row2: now reaches U1.36 (PF7)
- net Col0: now reaches U1.37 (PF6)
- net Col1: now reaches U1.38 (PF5)
- net Row3: now reaches U1.39 (PF4)
- net Row4: now reaches U1.40 (PF1)
- net Col3: now reaches U1.41 (PF0)
Changed lines of the file:
@@
 	0    1    1    0
+$EndComp
+$Comp
+L power:GND #PWR0102
+U 1 1 6228E976
+P 2400 7450
+F 0 "#PWR0102" H 2400 7200 50  0001 C CNN
+F 1 "GND" H 2405 7277 50  0000 C CNN
+F 2 "" H 2400 7450 50  0001 C CNN
+F 3 "" H 2400 7450 50  0001 C CNN
+	1    2400 7450
+	1    0    0    -1
+$EndComp
+Wire Wire Line
+	2750 3700 2750 3850
+$Comp
+L power:+5V #PWR0101
+U 1 1 622836F5
+P 2750 3700
+F 0 "#PWR0101" H 2750 3550 50  0001 C CNN
+F 1 "+5V" H 2765 3873 50  0000 C CNN
+F 2 "" H 2750 3700 50  0001 C CNN
+F 3 "" H 2750 3700 50  0001 C CNN
+	1    2750 3700
+	1    0    0    -1
+$EndComp
+$Sheet
+S 9500 4950 1600 1450
+U 62363975
+F0 "switch matrix" 50
+F1 "matrix.sch" 50
+$EndSheet
+$Comp
+L Connector_Generic:Conn_01x04 J1
+U 1 1 626DFEAA
+P 1400 2250
+F 0 "J1" H 1480 2242 50  0000 L CNN
+F 1 "Conn_01x04" H 1480 2151 50  0000 L CNN
+F 2 "random-keyboard-parts:JST-SR-4" H 1400 2250 50  0001 C CNN
+F 3 "~" H 1400 2250 50  0001 C CNN
+	1    1400 2250
+	1    0    0    -1
+$EndComp
+Wire Wire Line
+	1200 2150 1050 2150
+Wire Wire Line
+	1050 2150 1050 2050
+$Comp
+L power:VBUS #PWR0111
+U 1 1 626E380F
+P 1050 2050
+F 0 "#PWR0111" H 1050 1900 50  0001 C CNN
+F 1 "VBUS" H 1065 2223 50  0000 C CNN
+F 2 "" H 1050 2050 50  0001 C CNN
+F 3 "" H 1050 2050 50  0001 C CNN
+	1    1050 2050
+	1    0    0    -1
+$EndComp
+Wire Wire Line
+	1200 2450 1050 2450
+Wire Wire Line
+	1050 2450 1050 2550
+$Comp
+L power:GND #PWR0112
+U 1 1 626E5F38
+P 1050 2550
+F 0 "#PWR0112" H 1050 2300 50  0001 C CNN
+F 1 "GND" H 1055 2377 50  0000 C CNN
+F 2 "" H 1050 2550 50  0001 C CNN
+F 3 "" H 1050 2550 50  0001 C CNN
+	1    1050 2550
+	1    0    0    -1
+$EndComp
+Wire Wire Line
+	1200 2350 1050 2350
+Wire Wire Line
+	1200 2250 1050 2250
+Text GLabel 1050 2250 0    50   Input ~ 0
+D-
+Text GLabel 1050 2350 0    50   Input ~ 0
+D+
+$Comp
+L Power_Protection:SRV05-4 U2
+U 1 1 6234A89E
+P 3300 1800
+F 0 "U2" H 3300 2481 50  0000 C CNN
+F 1 "SRV05-4" H 3300 2390 50  0000 C CNN
+F 2 "Package_TO_SOT_SMD:SOT-23-6" H 4000 1350 50  0001 C CNN
+F 3 "http://www.onsemi.com/pub/Collateral/SRV05-4-D.PDF" H 3300 1800 50  0001 C CNN
+	1    3300 1800
+	1    0    0    -1
+$EndComp
+NoConn ~ 3800 1700
+NoConn ~ 2800 1900
+Wire Wire Line
+	2800 1700 2650 1700
+Wire Wire Line
+	3800 1900 3950 1900
+Text GLabel 2650 1700 0    50   Input ~ 0
+D+
+Text GLabel 3950 1900 2    50   Input ~ 0
+D-
+Wire Wire Line
+	3300 2300 3550 2300
+$Comp
+L power:GND #PWR0113
+U 1 1 623564EB
+P 3550 2300
+F 0 "#PWR0113" H 3550 2050 50  0001 C CNN
+F 1 "GND" H 3555 2127 50  0000 C CNN
+F 2 "" H 3550 2300 50  0001 C CNN
+F 3 "" H 3550 2300 50  0001 C CNN
+	1    3550 2300
+	1    0    0    -1
+$EndComp
+Wire Wire Line
+	3300 1300 3550 1300
+$Comp
+L power:VBUS #PWR0114
+U 1 1 6235878A
+P 3550 1300
+F 0 "#PWR0114" H 3550 1150 50  0001 C CNN
+F 1 "VBUS" H 3565 1473 50  0000 C CNN
+F 2 "" H 3550 1300 50  0001 C CNN
+F 3 "" H 3550 1300 50  0001 C CNN
+	1    3550 1300
+	1    0    0    -1
+$EndComp
+Text GLabel 3450 5450 2    50   Input ~ 0
+Col15
+Text GLabel 3450 5550 2    50   Input ~ 0
+Col14
+Text GLabel 3450 5650 2    50   Input ~ 0
+Col13
+Text GLabel 3450 5750 2    50   Input ~ 0
+Col11
+Text GLabel 3450 5950 2    50   Input ~ 0
+Col10
+Text GLabel 3450 6050 2    50   Input ~ 0
+Col9
+Text GLabel 3450 5850 2    50   Input ~ 0
+Col12
+Connection ~ 2750 3850
+Wire Wire Line
+	2750 3850 2850 3850
+Wire Wire Line
+	2850 3850 2950 3850
+Connection ~ 2850 3850
+Wire Wire Line
+	2400 7450 2750 7450
+Wire Wire Line
+	2750 7450 2850 7450
+Connection ~ 2750 7450
+$Comp
+L MCU_Microchip_ATmega:ATmega32U4-AU U1
+U 1 1 6227D02D
+P 2850 5650
+F 0 "U1" H 2850 3761 50  0000 C CNN
+F 1 "ATmega32U4-AU" H 2850 3670 50  0000 C CNN
+F 2 "Package_QFP:TQFP-44_10x10mm_P0.8mm" H 2850 5650 50  0001 C CIN
+F 3 "http://ww1.microchip.com/downloads/en/DeviceDoc/Atmel-7766-8-bit-AVR-ATmega16U4-32U4_Datasheet.pdf" H 2850 5650 50  0001 C CNN
+	1    2850 5650
+	1    0    0    -1
 $EndComp
 Wire Wire Line
@@
 	0    1    1    0
 $EndComp
-Connection ~ 2750 7450
-Wire Wire Line
-	2750 7450 2850 7450
-Wire Wire Line
-	2400 7450 2750 7450
-$Comp
-L power:GND #PWR0102
-U 1 1 6228E976
-P 2400 7450
-F 0 "#PWR0102" H 2400 7200 50  0001 C CNN
-F 1 "GND" H 2405 7277 50  0000 C CNN
-F 2 "" H 2400 7450 50  0001 C CNN
-F 3 "" H 2400 7450 50  0001 C CNN
-	1    2400 7450
-	1    0    0    -1
-$EndComp
-Connection ~ 2850 3850
-Wire Wire Line
-	2850 3850 2950 3850
-Connection ~ 2750 3850
-Wire Wire Line
-	2750 3850 2850 3850
-Wire Wire Line
-	2750 3700 2750 3850
-$Comp
-L power:+5V #PWR0101
-U 1 1 622836F5
-P 2750 3700
-F 0 "#PWR0101" H 2750 3550 50  0001 C CNN
-F 1 "+5V" H 2765 3873 50  0000 C CNN
-F 2 "" H 2750 3700 50  0001 C CNN
-F 3 "" H 2750 3700 50  0001 C CNN
-	1    2750 3700
-	1    0    0    -1
-$EndComp
-$Comp
-L MCU_Microchip_ATmega:ATmega32U4-AU U1
-U 1 1 6227D02D
-P 2850 5650
-F 0 "U1" H 2850 3761 50  0000 C CNN
-F 1 "ATmega32U4-AU" H 2850 3670 50  0000 C CNN
-F 2 "Package_QFP:TQFP-44_10x10mm_P0.8mm" H 2850 5650 50  0001 C CIN
-F 3 "http://ww1.microchip.com/downloads/en/DeviceDoc/Atmel-7766-8-bit-AVR-ATmega16U4-32U4_Datasheet.pdf" H 2850 5650 50  0001 C CNN
-	1    2850 5650
-	1    0    0    -1
-$EndComp
-$Sheet
-S 9500 4950 1600 1450
-U 62363975
-F0 "switch matrix" 50
-F1 "matrix.sch" 50
-$EndSheet
-$Comp
-L Connector_Generic:Conn_01x04 J1
-U 1 1 626DFEAA
-P 1400 2250
-F 0 "J1" H 1480 2242 50  0000 L CNN
-F 1 "Conn_01x04" H 1480 2151 50  0000 L CNN
-F 2 "random-keyboard-parts:JST-SR-4" H 1400 2250 50  0001 C CNN
-F 3 "~" H 1400 2250 50  0001 C CNN
-	1    1400 2250
-	1    0    0    -1
-$EndComp
-Wire Wire Line
-	1200 2150 1050 2150
-Wire Wire Line
-	1050 2150 1050 2050
-$Comp
-L power:VBUS #PWR0111
-U 1 1 626E380F
-P 1050 2050
-F 0 "#PWR0111" H 1050 1900 50  0001 C CNN
-F 1 "VBUS" H 1065 2223 50  0000 C CNN
-F 2 "" H 1050 2050 50  0001 C CNN
-F 3 "" H 1050 2050 50  0001 C CNN
-	1    1050 2050
-	1    0    0    -1
-$EndComp
-Wire Wire Line
-	1200 2450 1050 2450
-Wire Wire Line
-	1050 2450 1050 2550
-$Comp
-L power:GND #PWR0112
-U 1 1 626E5F38
-P 1050 2550
-F 0 "#PWR0112" H 1050 2300 50  0001 C CNN
-F 1 "GND" H 1055 2377 50  0000 C CNN
-F 2 "" H 1050 2550 50  0001 C CNN
-F 3 "" H 1050 2550 50  0001 C CNN
-	1    1050 2550
-	1    0    0    -1
-$EndComp
-Wire Wire Line
-	1200 2350 1050 2350
-Wire Wire Line
-	1200 2250 1050 2250
-Text GLabel 1050 2250 0    50   Input ~ 0
-D-
-Text GLabel 1050 2350 0    50   Input ~ 0
-D+
-$Comp
-L Power_Protection:SRV05-4 U2
-U 1 1 6234A89E
-P 3300 1800
-F 0 "U2" H 3300 2481 50  0000 C CNN
-F 1 "SRV05-4" H 3300 2390 50  0000 C CNN
-F 2 "Package_TO_SOT_SMD:SOT-23-6" H 4000 1350 50  0001 C CNN
-F 3 "http://www.onsemi.com/pub/Collateral/SRV05-4-D.PDF" H 3300 1800 50  0001 C CNN
-	1    3300 1800
-	1    0    0    -1
-$EndComp
-NoConn ~ 3800 1700
-NoConn ~ 2800 1900
-Wire Wire Line
-	2800 1700 2650 1700
-Wire Wire Line
-	3800 1900 3950 1900
-Text GLabel 2650 1700 0    50   Input ~ 0
-D+
-Text GLabel 3950 1900 2    50   Input ~ 0
-D-
-Wire Wire Line
-	3300 2300 3550 2300
-$Comp
-L power:GND #PWR0113
-U 1 1 623564EB
-P 3550 2300
-F 0 "#PWR0113" H 3550 2050 50  0001 C CNN
-F 1 "GND" H 3555 2127 50  0000 C CNN
-F 2 "" H 3550 2300 50  0001 C CNN
-F 3 "" H 3550 2300 50  0001 C CNN
-	1    3550 2300
-	1    0    0    -1
-$EndComp
-Wire Wire Line
-	3300 1300 3550 1300
-$Comp
-L power:VBUS #PWR0114
-U 1 1 6235878A
-P 3550 1300
-F 0 "#PWR0114" H 3550 1150 50  0001 C CNN
-F 1 "VBUS" H 3565 1473 50  0000 C CNN
-F 2 "" H 3550 1300 50  0001 C CNN
-F 3 "" H 3550 1300 50  0001 C CNN
-	1    3550 1300
-	1    0    0    -1
-$EndComp
+Text GLabel 3450 6350 2    50   Input ~ 0
+Row0
+Text GLabel 3450 4550 2    50   Input ~ 0
+Col8
+Text GLabel 3450 5350 2    50   Input ~ 0
+Col16
+Text GLabel 3450 4650 2    50   Input ~ 0
+Col7
+Text GLabel 3450 4750 2    50   Input ~ 0
+Col6
+Text GLabel 3450 5050 2    50   Input ~ 0
+Col5
+Text GLabel 3450 5150 2    50   Input ~ 0
+Col4
+Text GLabel 3450 7050 2    50   Input ~ 0
+Row2
+Text GLabel 3450 6550 2    50   Input ~ 0
+Col3
+Text GLabel 3450 4850 2    50   Input ~ 0
+Row1
+Text GLabel 3450 6950 2    50   Input ~ 0
+Col0
+Text GLabel 3450 6850 2    50   Input ~ 0
+Col1
+Text GLabel 3450 6750 2    50   Input ~ 0
+Row3
+Text GLabel 3450 6650 2    50   Input ~ 0
+Row4
 $EndSCHEMATC
