File: attempt2-pcb.sch (KiCad schematic (older format))
At the start: 16 parts, among them J1 Conn_01x04, SW1 SW_Push, U1 ATmega32U4-AU, U2 SRV05-4, Y1 16MHz

Commit message: proofing
Parts:
- SW1: value SW_Push -> Reset
Connections:
- net Col2: now reaches U1.10 (PB2)
- net Reset: now reaches R1.2, SW1.2, U1.13 (~RESET)
- net XTAL2: now reaches C2.1, U1.16 (XTAL2), Y1.3
- net XTAL1: now reaches C1.1, U1.17 (XTAL1), Y1.1
- net MCU_D-: now reaches R3.1, U1.3 (D-)
- net MCU_D+: now reaches R2.1, U1.4 (D+)
- no-connect marks 2 -> 3
Other:
- moved on the sheet: C1, C2, R1, SW1, Y1
Changed lines of the file:
@@
 Wire Wire Line
 	3900 6250 4200 6250
-Text GLabel 700  5150 0    50   Input ~ 0
-D+
-Text GLabel 700  5250 0    50   Input ~ 0
-D-
-Wire Wire Line
-	2150 3600 2150 3700
+Wire Wire Line
+	1550 3600 1550 3700
 $Comp
 L power:+5V #PWR0110
 U 1 1 622EE29C
-P 2150 3600
-F 0 "#PWR0110" H 2150 3450 50  0001 C CNN
-F 1 "+5V" H 2165 3773 50  0000 C CNN
-F 2 "" H 2150 3600 50  0001 C CNN
-F 3 "" H 2150 3600 50  0001 C CNN
-	1    2150 3600
-	1    0    0    -1
-$EndComp
-Wire Wire Line
-	2150 4150 2250 4150
-Connection ~ 2150 4150
-Wire Wire Line
-	2150 3900 2150 4150
+P 1550 3600
+F 0 "#PWR0110" H 1550 3450 50  0001 C CNN
+F 1 "+5V" H 1565 3773 50  0000 C CNN
+F 2 "" H 1550 3600 50  0001 C CNN
+F 3 "" H 1550 3600 50  0001 C CNN
+	1    1550 3600
+	1    0    0    -1
+$EndComp
+Wire Wire Line
+	1550 4150 1650 4150
+Connection ~ 1550 4150
+Wire Wire Line
+	1550 3900 1550 4150
 $Comp
 L Device:R_Small R1
 U 1 1 622EC068
-P 2150 3800
-F 0 "R1" H 2209 3846 50  0000 L CNN
-F 1 "10k" H 2209 3755 50  0000 L CNN
-F 2 "Resistor_SMD:R_0805_2012Metric" H 2150 3800 50  0001 C CNN
-F 3 "~" H 2150 3800 50  0001 C CNN
-	1    2150 3800
-	1    0    0    -1
-$EndComp
-Wire Wire Line
-	2050 4150 2150 4150
-Wire Wire Line
-	1650 4050 1650 4150
-Wire Wire Line
-	1500 4050 1650 4050
+P 1550 3800
+F 0 "R1" H 1609 3846 50  0000 L CNN
+F 1 "10k" H 1609 3755 50  0000 L CNN
+F 2 "Resistor_SMD:R_0805_2012Metric" H 1550 3800 50  0001 C CNN
+F 3 "~" H 1550 3800 50  0001 C CNN
+	1    1550 3800
+	1    0    0    -1
+$EndComp
+Wire Wire Line
+	1450 4150 1550 4150
+Wire Wire Line
+	1050 4050 1050 4150
+Wire Wire Line
+	900  4050 1050 4050
 $Comp
 L power:GND #PWR0109
 U 1 1 622E75BF
-P 1500 4050
-F 0 "#PWR0109" H 1500 3800 50  0001 C CNN
-F 1 "GND" H 1505 3877 50  0000 C CNN
-F 2 "" H 1500 4050 50  0001 C CNN
-F 3 "" H 1500 4050 50  0001 C CNN
-	1    1500 4050
+P 900 4050
+F 0 "#PWR0109" H 900 3800 50  0001 C CNN
+F 1 "GND" H 905 3877 50  0000 C CNN
+F 2 "" H 900 4050 50  0001 C CNN
+F 3 "" H 900 4050 50  0001 C CNN
+	1    900  4050
 	1    0    0    -1
 $EndComp
@@
 L Switch:SW_Push SW1
 U 1 1 622E5F62
-P 1850 4150
-F 0 "SW1" H 1850 4435 50  0000 C CNN
-F 1 "SW_Push" H 1850 4344 50  0000 C CNN
-F 2 "random-keyboard-parts:SKQG-1155865" H 1850 4350 50  0001 C CNN
-F 3 "~" H 1850 4350 50  0001 C CNN
-	1    1850 4150
-	1    0    0    -1
-$EndComp
-Wire Wire Line
-	1700 4700 1700 4750
-Connection ~ 1700 4700
-Wire Wire Line
-	1900 4700 1700 4700
-Wire Wire Line
-	1900 4450 1900 4700
-Connection ~ 1200 4750
-Wire Wire Line
-	1700 4450 1700 4700
-Wire Wire Line
-	1700 4750 1200 4750
-Connection ~ 1200 4600
-Wire Wire Line
-	1200 4600 1200 4750
-Wire Wire Line
-	1200 4300 1200 4600
+P 1250 4150
+F 0 "SW1" H 1250 4435 50  0000 C CNN
+F 1 "Reset" H 1250 4344 50  0000 C CNN
+F 2 "random-keyboard-parts:SKQG-1155865" H 1250 4350 50  0001 C CNN
+F 3 "~" H 1250 4350 50  0001 C CNN
+	1    1250 4150
+	1    0    0    -1
+$EndComp
+Wire Wire Line
+	1100 4700 1100 4750
+Connection ~ 1100 4700
+Wire Wire Line
+	1300 4700 1100 4700
+Wire Wire Line
+	1300 4450 1300 4700
+Connection ~ 600  4750
+Wire Wire Line
+	1100 4450 1100 4700
+Wire Wire Line
+	1100 4750 600  4750
+Connection ~ 600  4600
+Wire Wire Line
+	600  4600 600  4750
+Wire Wire Line
+	600  4300 600  4600
 $Comp
 L power:GND #PWR0108
 U 1 1 622D8F6E
-P 1200 4750
-F 0 "#PWR0108" H 1200 4500 50  0001 C CNN
-F 1 "GND" H 1205 4577 50  0000 C CNN
-F 2 "" H 1200 4750 50  0001 C CNN
-F 3 "" H 1200 4750 50  0001 C CNN
-	1    1200 4750
-	1    0    0    -1
-$EndComp
-Connection ~ 1800 4350
-Wire Wire Line
-	1800 4300 1800 4350
-Wire Wire Line
-	1400 4300 1800 4300
-Connection ~ 1800 4550
-Wire Wire Line
-	1800 4600 1800 4550
-Wire Wire Line
-	1400 4600 1800 4600
+P 600 4750
+F 0 "#PWR0108" H 600 4500 50  0001 C CNN
+F 1 "GND" H 605 4577 50  0000 C CNN
+F 2 "" H 600 4750 50  0001 C CNN
+F 3 "" H 600 4750 50  0001 C CNN
+	1    600  4750
+	1    0    0    -1
+$EndComp
+Wire Wire Line
+	1200 4300 1200 4350
+Wire Wire Line
+	800  4300 1200 4300
+Wire Wire Line
+	1200 4600 1200 4550
+Wire Wire Line
+	800  4600 1200 4600
 $Comp
 L Device:C_Small C2
 U 1 1 622D720B
-P 1300 4600
-F 0 "C2" V 1071 4600 50  0000 C CNN
-F 1 "22pF" V 1162 4600 50  0000 C CNN
-F 2 "Capacitor_SMD:C_0805_2012Metric" H 1300 4600 50  0001 C CNN
-F 3 "~" H 1300 4600 50  0001 C CNN
-	1    1300 4600
+P 700 4600
+F 0 "C2" V 471 4600 50  0000 C CNN
+F 1 "22pF" V 562 4600 50  0000 C CNN
+F 2 "Capacitor_SMD:C_0805_2012Metric" H 700 4600 50  0001 C CNN
+F 3 "~" H 700 4600 50  0001 C CNN
+	1    700  4600
 	0    1    1    0
 $EndComp
@@
 L Device:C_Small C1
 U 1 1 622D5727
-P 1300 4300
-F 0 "C1" V 1071 4300 50  0000 C CNN
-F 1 "22pF" V 1162 4300 50  0000 C CNN
-F 2 "Capacitor_SMD:C_0805_2012Metric" H 1300 4300 50  0001 C CNN
-F 3 "~" H 1300 4300 50  0001 C CNN
-	1    1300 4300
+P 700 4300
+F 0 "C1" V 471 4300 50  0000 C CNN
+F 1 "22pF" V 562 4300 50  0000 C CNN
+F 2 "Capacitor_SMD:C_0805_2012Metric" H 700 4300 50  0001 C CNN
+F 3 "~" H 700 4300 50  0001 C CNN
+	1    700  4300
 	0    1    1    0
 $EndComp
 Wire Wire Line
-	1800 4550 2250 4550
-Wire Wire Line
-	1800 4350 2250 4350
+	1200 4550 1650 4550
+Wire Wire Line
+	1200 4350 1650 4350
 $Comp
 L Device:Crystal_GND24_Small Y1
 U 1 1 622D2674
-P 1800 4450
-F 0 "Y1" V 1754 4594 50  0000 L CNN
-F 1 "16MHz" V 1845 4594 50  0000 L CNN
-F 2 "Crystal:Crystal_SMD_3225-4Pin_3.2x2.5mm" H 1800 4450 50  0001 C CNN
-F 3 "~" H 1800 4450 50  0001 C CNN
-	1    1800 4450
+P 1200 4450
+F 0 "Y1" V 1154 4594 50  0000 L CNN
+F 1 "16MHz" V 1245 4594 50  0000 L CNN
+F 2 "Crystal:Crystal_SMD_3225-4Pin_3.2x2.5mm" H 1200 4450 50  0001 C CNN
+F 3 "~" H 1200 4450 50  0001 C CNN
+	1    1200 4450
 	0    1    1    0
 $EndComp
@@
 	1    1650 5550
 	1    0    0    -1
-$EndComp
-Wire Wire Line
-	1400 5150 700  5150
-Wire Wire Line
-	1050 5250 700  5250
-Wire Wire Line
-	1250 5250 2250 5250
-Wire Wire Line
-	1600 5150 2250 5150
-$Comp
-L Device:R_Small R3
-U 1 1 622967D3
-P 1150 5250
-F 0 "R3" V 954 5250 50  0000 C CNN
-F 1 "22" V 1045 5250 50  0000 C CNN
-F 2 "Resistor_SMD:R_0805_2012Metric" H 1150 5250 50  0001 C CNN
-F 3 "~" H 1150 5250 50  0001 C CNN
-	1    1150 5250
-	0    1    1    0
-$EndComp
-$Comp
-L Device:R_Small R2
-U 1 1 6229476D
-P 1500 5150
-F 0 "R2" V 1304 5150 50  0000 C CNN
-F 1 "22" V 1395 5150 50  0000 C CNN
-F 2 "Resistor_SMD:R_0805_2012Metric" H 1500 5150 50  0001 C CNN
-F 3 "~" H 1500 5150 50  0001 C CNN
-	1    1500 5150
-	0    1    1    0
 $EndComp
 $Comp
@@
 Text GLabel 3450 6650 2    50   Input ~ 0
 Row4
+Text GLabel 3450 4350 2    50   Input ~ 0
+Col2
+Text GLabel 1650 4150 2    50   Input ~ 0
+Reset
+Text GLabel 2250 4150 0    50   Input ~ 0
+Reset
+Connection ~ 1200 4350
+Connection ~ 1200 4550
+Text GLabel 2250 4350 0    50   Input ~ 0
+XTAL1
+Text GLabel 2250 4550 0    50   Input ~ 0
+XTAL2
+Text GLabel 1650 4350 2    50   Input ~ 0
+XTAL1
+Text GLabel 1650 4550 2    50   Input ~ 0
+XTAL2
+NoConn ~ 2250 4750
+$Comp
+L Device:R_Small R2
+U 1 1 6229476D
+P 1500 5150
+F 0 "R2" V 1304 5150 50  0000 C CNN
+F 1 "22" V 1395 5150 50  0000 C CNN
+F 2 "Resistor_SMD:R_0805_2012Metric" H 1500 5150 50  0001 C CNN
+F 3 "~" H 1500 5150 50  0001 C CNN
+	1    1500 5150
+	0    1    1    0
+$EndComp
+$Comp
+L Device:R_Small R3
+U 1 1 622967D3
+P 1150 5250
+F 0 "R3" V 954 5250 50  0000 C CNN
+F 1 "22" V 1045 5250 50  0000 C CNN
+F 2 "Resistor_SMD:R_0805_2012Metric" H 1150 5250 50  0001 C CNN
+F 3 "~" H 1150 5250 50  0001 C CNN
+	1    1150 5250
+	0    1    1    0
+$EndComp
+Wire Wire Line
+	1600 5150 2250 5150
+Wire Wire Line
+	1250 5250 2250 5250
+Wire Wire Line
+	1050 5250 700  5250
+Wire Wire Line
+	1400 5150 700  5150
+Text GLabel 700  5250 0    50   Input ~ 0
+D-
+Text GLabel 700  5150 0    50   Input ~ 0
+D+
+Text Label 2100 5150 2    50   ~ 0
+MCU_D+
+Text Label 2100 5250 2    50   ~ 0
+MCU_D-
 $EndSCHEMATC

Commit message: Big Changes
Parts:
- removed U1: ATmega32U4-AU, Package_QFP:TQFP-44_10x10mm_P0.8mm, symbol MCU_Microchip_ATmega:ATmega32U4-AU
- added U1: ATmega32U4-MU, Package_DFN_QFN:QFN-44-1EP_7x7mm_P0.5mm_EP5.2x5.2mm, symbol MCU_Microchip_ATmega:ATmega32U4-MU
Connections:
- net +5V: now also U1.14 (VCC), U1.2 (UVCC), U1.24 (AVCC), U1.34 (VCC), U1.44 (AVCC), U1.7 (VBUS)
- net Col0: now also U1.37 (PF6)
- net Col1: now also U1.38 (PF5)
- net Col10: now also U1.26 (PD6)
- net Col11: now also U1.25 (PD4)
- net Col12: now also U1.22 (PD5)
- net Col13: now also U1.21 (PD3)
- net Col14: now also U1.20 (PD2)
- net Col15: now also U1.19 (PD1)
- net Col16: now also U1.18 (PD0)
- net Col2: now also U1.10 (PB2)
- net Col3: now also U1.41 (PF0)
- net Col4: now also U1.32 (PC7)
- net Col5: now also U1.31 (PC6)
- net Col6: now also U1.30 (PB6)
- net Col7: now also U1.29 (PB5)
- net Col8: now also U1.28 (PB4)
- net Col9: now also U1.27 (PD7)
- net GND: now also U1.15 (GND), U1.23 (GND), U1.35 (GND), U1.43 (GND), U1.45 (GND), U1.5 (UGND)
- net MCU_D+: now also U1.4 (D+)
- net MCU_D-: now also U1.3 (D-)
- net Reset: now also U1.13 (~RESET)
- net Row0: now also U1.1 (PE6)
- net Row1: now also U1.12 (PB7)
- net Row2: now also U1.36 (PF7)
- net Row3: now also U1.39 (PF4)
- net Row4: now also U1.40 (PF1)
- net XTAL1: now also U1.17 (XTAL1)
- net XTAL2: now also U1.16 (XTAL2)
- net at R4.2: now also U1.33 (~HWB~/PE2)
- net at C3.1: now also U1.6 (UCAP)
Changed lines of the file:
@@
 Text GLabel 3450 5850 2    50   Input ~ 0
 Col12
-Connection ~ 2750 3850
-Wire Wire Line
-	2750 3850 2850 3850
-Wire Wire Line
-	2850 3850 2950 3850
-Connection ~ 2850 3850
-Wire Wire Line
-	2400 7450 2750 7450
-Wire Wire Line
-	2750 7450 2850 7450
-Connection ~ 2750 7450
-$Comp
-L MCU_Microchip_ATmega:ATmega32U4-AU U1
-U 1 1 6227D02D
-P 2850 5650
-F 0 "U1" H 2850 3761 50  0000 C CNN
-F 1 "ATmega32U4-AU" H 2850 3670 50  0000 C CNN
-F 2 "Package_QFP:TQFP-44_10x10mm_P0.8mm" H 2850 5650 50  0001 C CIN
-F 3 "http://ww1.microchip.com/downloads/en/DeviceDoc/Atmel-7766-8-bit-AVR-ATmega16U4-32U4_Datasheet.pdf" H 2850 5650 50  0001 C CNN
-	1    2850 5650
-	1    0    0    -1
-$EndComp
 Wire Wire Line
 	3450 6250 3700 6250
@@
 Text Label 2100 5250 2    50   ~ 0
 MCU_D-
+$Comp
+L MCU_Microchip_ATmega:ATmega32U4-MU U1
+U 1 1 623FA336
+P 2850 5650
+F 0 "U1" H 2850 3761 50  0000 C CNN
+F 1 "ATmega32U4-MU" H 2850 3670 50  0000 C CNN
+F 2 "Package_DFN_QFN:QFN-44-1EP_7x7mm_P0.5mm_EP5.2x5.2mm" H 2850 5650 50  0001 C CIN
+F 3 "http://ww1.microchip.com/downloads/en/DeviceDoc/Atmel-7766-8-bit-AVR-ATmega16U4-32U4_Datasheet.pdf" H 2850 5650 50  0001 C CNN
+	1    2850 5650
+	1    0    0    -1
+$EndComp
+Wire Wire Line
+	2750 3850 2850 3850
+Wire Wire Line
+	2400 7450 2750 7450
+Connection ~ 2750 3850
+Wire Wire Line
+	2950 3850 2850 3850
+Connection ~ 2850 3850
+Wire Wire Line
+	2850 7450 2750 7450
+Connection ~ 2750 7450
 $EndSCHEMATC
